File: мой вариант часов/схема часов/file5F6C9CBF.sch (KiCad schematic (older format))
At the start: 14 parts

Commit message: version-1
Parts:
- BT1: renamed from BT?; footprint (none) -> TestPoint:TestPoint_Bridge_Pitch6.35mm_Drill1.3mm
- C1, C2: renamed from C?; footprint (none) -> TestPoint:TestPoint_2Pads_Pitch2.54mm_Drill0.8mm
- CB1: renamed from CB?; footprint (none) -> Button_Switch_THT:SW_PUSH_6mm_H9.5mm
- R1, R2, R3, R4, R5: renamed from R?; footprint (none) -> Diode_THT:D_A-405_P10.16mm_Horizontal
- gave numbers to parts that had none: 5
Connections:
- net Vo renamed Vout
- net постоянка_мк renamed KEY_V_MK
- net тип_питания renamed TYPE_V
Changed lines of the file:
@@
 $Descr A4 11693 8268
 encoding utf-8
-Sheet 2 4
+Sheet 2 6
 Title ""
 Date ""
@@
 P 1650 2800
 AR Path="/5F6E2D20" Ref="BT?"  Part="1"
-AR Path="/5F6C9CC0/5F6E2D20" Ref="BT?"  Part="1"
-F 0 "BT?" H 1768 2896 50  0000 L CNN
+AR Path="/5F6C9CC0/5F6E2D20" Ref="BT1"  Part="1"
+F 0 "BT1" H 1768 2896 50  0000 L CNN
 F 1 "Battery_Cell" H 1768 2805 50  0000 L CNN
-F 2 "" V 1650 2860 50  0001 C CNN
+F 2 "TestPoint:TestPoint_Bridge_Pitch6.35mm_Drill1.3mm" V 1650 2860 50  0001 C CNN
 F 3 "~" V 1650 2860 50  0001 C CNN
 	1    1650 2800
@@
 P 1650 2900
 AR Path="/5F6E2D26" Ref="#PWR?"  Part="1"
-AR Path="/5F6C9CC0/5F6E2D26" Ref="#PWR?"  Part="1"
-F 0 "#PWR?" H 1650 2650 50  0001 C CNN
+AR Path="/5F6C9CC0/5F6E2D26" Ref="#PWR0101"  Part="1"
+F 0 "#PWR0101" H 1650 2650 50  0001 C CNN
 F 1 "GND" H 1655 2727 50  0000 C CNN
 F 2 "" H 1650 2900 50  0001 C CNN
@@
 P 2500 2700
 AR Path="/5F6E2D2C" Ref="Q?"  Part="1"
-AR Path="/5F6C9CC0/5F6E2D2C" Ref="Q?"  Part="1"
-F 0 "Q?" V 2842 2700 50  0000 C CNN
+AR Path="/5F6C9CC0/5F6E2D2C" Ref="Q1"  Part="1"
+F 0 "Q1" V 2842 2700 50  0000 C CNN
 F 1 "IRLML6402" V 2751 2700 50  0000 C CNN
 F 2 "Package_TO_SOT_SMD:SOT-23" H 2700 2625 50  0001 L CIN
@@
 P 3050 2700
 AR Path="/5F6E2D32" Ref="Q?"  Part="1"
-AR Path="/5F6C9CC0/5F6E2D32" Ref="Q?"  Part="1"
-F 0 "Q?" V 3392 2700 50  0000 C CNN
+AR Path="/5F6C9CC0/5F6E2D32" Ref="Q3"  Part="1"
+F 0 "Q3" V 3392 2700 50  0000 C CNN
 F 1 "IRLML6402" V 3301 2700 50  0000 C CNN
 F 2 "Package_TO_SOT_SMD:SOT-23" H 3250 2625 50  0001 L CIN
@@
 P 2200 2750
 AR Path="/5F6E2D3B" Ref="R?"  Part="1"
-AR Path="/5F6C9CC0/5F6E2D3B" Ref="R?"  Part="1"
-F 0 "R?" H 2270 2796 50  0000 L CNN
+AR Path="/5F6C9CC0/5F6E2D3B" Ref="R2"  Part="1"
+F 0 "R2" H 2270 2796 50  0000 L CNN
 F 1 "200k " H 2270 2705 50  0000 L CNN
-F 2 "" V 2130 2750 50  0001 C CNN
+F 2 "Diode_THT:D_A-405_P10.16mm_Horizontal" V 2130 2750 50  0001 C CNN
 F 3 "~" H 2200 2750 50  0001 C CNN
 	1    2200 2750
@@
 P 3750 1950
 AR Path="/5F6E2D49" Ref="D?"  Part="1"
-AR Path="/5F6C9CC0/5F6E2D49" Ref="D?"  Part="1"
-F 0 "D?" V 3704 2038 50  0000 L CNN
+AR Path="/5F6C9CC0/5F6E2D49" Ref="D1"  Part="1"
+F 0 "D1" V 3704 2038 50  0000 L CNN
 F 1 "BAT54C" V 3795 2038 50  0000 L CNN
 F 2 "Package_TO_SOT_SMD:SOT-23" H 3825 2075 50  0001 L CNN
@@
 P 3750 2250
 AR Path="/5F6E2D4F" Ref="#PWR?"  Part="1"
-AR Path="/5F6C9CC0/5F6E2D4F" Ref="#PWR?"  Part="1"
-F 0 "#PWR?" H 3750 2000 50  0001 C CNN
+AR Path="/5F6C9CC0/5F6E2D4F" Ref="#PWR0102"  Part="1"
+F 0 "#PWR0102" H 3750 2000 50  0001 C CNN
 F 1 "GND" H 3755 2077 50  0000 C CNN
 F 2 "" H 3750 2250 50  0001 C CNN
@@
 P 3750 1650
 AR Path="/5F6E2D55" Ref="#PWR?"  Part="1"
-AR Path="/5F6C9CC0/5F6E2D55" Ref="#PWR?"  Part="1"
-F 0 "#PWR?" H 3750 1500 50  0001 C CNN
+AR Path="/5F6C9CC0/5F6E2D55" Ref="#PWR0103"  Part="1"
+F 0 "#PWR0103" H 3750 1500 50  0001 C CNN
 F 1 "+12C" H 3765 1823 50  0000 C CNN
 F 2 "" H 3750 1650 50  0001 C CNN
@@
 P 3050 3050
 AR Path="/5F6E2D5B" Ref="R?"  Part="1"
-AR Path="/5F6C9CC0/5F6E2D5B" Ref="R?"  Part="1"
-F 0 "R?" H 3120 3096 50  0000 L CNN
+AR Path="/5F6C9CC0/5F6E2D5B" Ref="R3"  Part="1"
+F 0 "R3" H 3120 3096 50  0000 L CNN
 F 1 "10k " H 3120 3005 50  0000 L CNN
-F 2 "" V 2980 3050 50  0001 C CNN
+F 2 "Diode_THT:D_A-405_P10.16mm_Horizontal" V 2980 3050 50  0001 C CNN
 F 3 "~" H 3050 3050 50  0001 C CNN
 	1    3050 3050
@@
 P 4500 1950
 AR Path="/5F6E2D61" Ref="D?"  Part="1"
-AR Path="/5F6C9CC0/5F6E2D61" Ref="D?"  Part="1"
-F 0 "D?" V 4454 2038 50  0000 L CNN
+AR Path="/5F6C9CC0/5F6E2D61" Ref="D2"  Part="1"
+F 0 "D2" V 4454 2038 50  0000 L CNN
 F 1 "BAT54C" V 4545 2038 50  0000 L CNN
 F 2 "Package_TO_SOT_SMD:SOT-23" H 4575 2075 50  0001 L CNN
@@
 P 4500 2250
 AR Path="/5F6E2D67" Ref="#PWR?"  Part="1"
-AR Path="/5F6C9CC0/5F6E2D67" Ref="#PWR?"  Part="1"
-F 0 "#PWR?" H 4500 2000 50  0001 C CNN
+AR Path="/5F6C9CC0/5F6E2D67" Ref="#PWR0104"  Part="1"
+F 0 "#PWR0104" H 4500 2000 50  0001 C CNN
 F 1 "GND" H 4505 2077 50  0000 C CNN
 F 2 "" H 4500 2250 50  0001 C CNN
@@
 P 4500 1650
 AR Path="/5F6E2D6D" Ref="#PWR?"  Part="1"
-AR Path="/5F6C9CC0/5F6E2D6D" Ref="#PWR?"  Part="1"
-F 0 "#PWR?" H 4500 1500 50  0001 C CNN
+AR Path="/5F6C9CC0/5F6E2D6D" Ref="#PWR0105"  Part="1"
+F 0 "#PWR0105" H 4500 1500 50  0001 C CNN
 F 1 "+12C" H 4515 1823 50  0000 C CNN
 F 2 "" H 4500 1650 50  0001 C CNN
@@
 P 4250 2750
 AR Path="/5F6E2D76" Ref="R?"  Part="1"
-AR Path="/5F6C9CC0/5F6E2D76" Ref="R?"  Part="1"
-F 0 "R?" H 4320 2796 50  0000 L CNN
+AR Path="/5F6C9CC0/5F6E2D76" Ref="R4"  Part="1"
+F 0 "R4" H 4320 2796 50  0000 L CNN
 F 1 "10k " H 4320 2705 50  0000 L CNN
-F 2 "" V 4180 2750 50  0001 C CNN
+F 2 "Diode_THT:D_A-405_P10.16mm_Horizontal" V 4180 2750 50  0001 C CNN
 F 3 "~" H 4250 2750 50  0001 C CNN
 	1    4250 2750
@@
 P 4250 3050
 AR Path="/5F6E2D7E" Ref="R?"  Part="1"
-AR Path="/5F6C9CC0/5F6E2D7E" Ref="R?"  Part="1"
-F 0 "R?" H 4320 3096 50  0000 L CNN
+AR Path="/5F6C9CC0/5F6E2D7E" Ref="R5"  Part="1"
+F 0 "R5" H 4320 3096 50  0000 L CNN
 F 1 "10k " H 4320 3005 50  0000 L CNN
-F 2 "" V 4180 3050 50  0001 C CNN
+F 2 "Diode_THT:D_A-405_P10.16mm_Horizontal" V 4180 3050 50  0001 C CNN
 F 3 "~" H 4250 3050 50  0001 C CNN
 	1    4250 3050
@@
 P 4250 3200
 AR Path="/5F6E2D84" Ref="#PWR?"  Part="1"
-AR Path="/5F6C9CC0/5F6E2D84" Ref="#PWR?"  Part="1"
-F 0 "#PWR?" H 4250 2950 50  0001 C CNN
+AR Path="/5F6C9CC0/5F6E2D84" Ref="#PWR0106"  Part="1"
+F 0 "#PWR0106" H 4250 2950 50  0001 C CNN
 F 1 "GND" H 4255 3027 50  0000 C CNN
 F 2 "" H 4250 3200 50  0001 C CNN
@@
 P 4600 3100
 AR Path="/5F6E2D8A" Ref="C?"  Part="1"
-AR Path="/5F6C9CC0/5F6E2D8A" Ref="C?"  Part="1"
-F 0 "C?" H 4715 3146 50  0000 L CNN
+AR Path="/5F6C9CC0/5F6E2D8A" Ref="C2"  Part="1"
+F 0 "C2" H 4715 3146 50  0000 L CNN
 F 1 "100n" H 4715 3055 50  0000 L CNN
-F 2 "" H 4638 2950 50  0001 C CNN
+F 2 "TestPoint:TestPoint_2Pads_Pitch2.54mm_Drill0.8mm" H 4638 2950 50  0001 C CNN
 F 3 "~" H 4600 3100 50  0001 C CNN
 	1    4600 3100
@@
 P 4600 3250
 AR Path="/5F6E2D93" Ref="#PWR?"  Part="1"
-AR Path="/5F6C9CC0/5F6E2D93" Ref="#PWR?"  Part="1"
-F 0 "#PWR?" H 4600 3000 50  0001 C CNN
+AR Path="/5F6C9CC0/5F6E2D93" Ref="#PWR0107"  Part="1"
+F 0 "#PWR0107" H 4600 3000 50  0001 C CNN
 F 1 "GND" H 4605 3077 50  0000 C CNN
 F 2 "" H 4600 3250 50  0001 C CNN
@@
 P 2550 3800
 AR Path="/5F6E2D9E" Ref="Q?"  Part="1"
-AR Path="/5F6C9CC0/5F6E2D9E" Ref="Q?"  Part="1"
-F 0 "Q?" H 2754 3846 50  0000 L CNN
+AR Path="/5F6C9CC0/5F6E2D9E" Ref="Q2"  Part="1"
+F 0 "Q2" H 2754 3846 50  0000 L CNN
 F 1 "BSS123" H 2754 3755 50  0000 L CNN
 F 2 "Package_TO_SOT_SMD:SOT-23" H 2750 3725 50  0001 L CIN
@@
 P 2650 4000
 AR Path="/5F6E2DA5" Ref="#PWR?"  Part="1"
-AR Path="/5F6C9CC0/5F6E2DA5" Ref="#PWR?"  Part="1"
-F 0 "#PWR?" H 2650 3750 50  0001 C CNN
+AR Path="/5F6C9CC0/5F6E2DA5" Ref="#PWR0108"  Part="1"
+F 0 "#PWR0108" H 2650 3750 50  0001 C CNN
 F 1 "GND" H 2655 3827 50  0000 C CNN
 F 2 "" H 2650 4000 50  0001 C CNN
@@
 P 2350 4650
 AR Path="/5F6E2DAE" Ref="CB?"  Part="1"
-AR Path="/5F6C9CC0/5F6E2DAE" Ref="CB?"  Part="1"
-F 0 "CB?" V 2085 4650 50  0000 C CNN
+AR Path="/5F6C9CC0/5F6E2DAE" Ref="CB1"  Part="1"
+F 0 "CB1" V 2085 4650 50  0000 C CNN
 F 1 "CircuitBreaker_1P" V 2176 4650 50  0000 C CNN
-F 2 "" H 2350 4650 50  0001 C CNN
+F 2 "Button_Switch_THT:SW_PUSH_6mm_H9.5mm" H 2350 4650 50  0001 C CNN
 F 3 "~" H 2350 4650 50  0001 C CNN
 	1    2350 4650
@@
 P 2700 4800
 AR Path="/5F6E2DB4" Ref="C?"  Part="1"
-AR Path="/5F6C9CC0/5F6E2DB4" Ref="C?"  Part="1"
-F 0 "C?" H 2815 4846 50  0000 L CNN
+AR Path="/5F6C9CC0/5F6E2DB4" Ref="C1"  Part="1"
+F 0 "C1" H 2815 4846 50  0000 L CNN
 F 1 "100n" H 2815 4755 50  0000 L CNN
-F 2 "" H 2738 4650 50  0001 C CNN
+F 2 "TestPoint:TestPoint_2Pads_Pitch2.54mm_Drill0.8mm" H 2738 4650 50  0001 C CNN
 F 3 "~" H 2700 4800 50  0001 C CNN
 	1    2700 4800
@@
 P 2700 4950
 AR Path="/5F6E2DBC" Ref="#PWR?"  Part="1"
-AR Path="/5F6C9CC0/5F6E2DBC" Ref="#PWR?"  Part="1"
-F 0 "#PWR?" H 2700 4700 50  0001 C CNN
+AR Path="/5F6C9CC0/5F6E2DBC" Ref="#PWR0109"  Part="1"
+F 0 "#PWR0109" H 2700 4700 50  0001 C CNN
 F 1 "GND" H 2705 4777 50  0000 C CNN
 F 2 "" H 2700 4950 50  0001 C CNN
@@
 P 2050 4650
 AR Path="/5F6E2DC2" Ref="#PWR?"  Part="1"
-AR Path="/5F6C9CC0/5F6E2DC2" Ref="#PWR?"  Part="1"
-F 0 "#PWR?" H 2050 4400 50  0001 C CNN
+AR Path="/5F6C9CC0/5F6E2DC2" Ref="#PWR0110"  Part="1"
+F 0 "#PWR0110" H 2050 4400 50  0001 C CNN
 F 1 "GND" H 2055 4477 50  0000 C CNN
 F 2 "" H 2050 4650 50  0001 C CNN
@@
 P 2150 3950
 AR Path="/5F6E2DC8" Ref="R?"  Part="1"
-AR Path="/5F6C9CC0/5F6E2DC8" Ref="R?"  Part="1"
-F 0 "R?" H 2220 3996 50  0000 L CNN
+AR Path="/5F6C9CC0/5F6E2DC8" Ref="R1"  Part="1"
+F 0 "R1" H 2220 3996 50  0000 L CNN
 F 1 "10k " H 2220 3905 50  0000 L CNN
-F 2 "" V 2080 3950 50  0001 C CNN
+F 2 "Diode_THT:D_A-405_P10.16mm_Horizontal" V 2080 3950 50  0001 C CNN
 F 3 "~" H 2150 3950 50  0001 C CNN
 	1    2150 3950
@@
 P 2150 4100
 AR Path="/5F6E2DD0" Ref="#PWR?"  Part="1"
-AR Path="/5F6C9CC0/5F6E2DD0" Ref="#PWR?"  Part="1"
-F 0 "#PWR?" H 2150 3850 50  0001 C CNN
+AR Path="/5F6C9CC0/5F6E2DD0" Ref="#PWR0111"  Part="1"
+F 0 "#PWR0111" H 2150 3850 50  0001 C CNN
 F 1 "GND" H 2155 3927 50  0000 C CNN
 F 2 "" H 2150 4100 50  0001 C CNN
@@
 	1    0    0    -1
 $EndComp
-Text GLabel 5450 2600 2    50   Input ~ 0
-Vo
-Text GLabel 1800 3800 0    50   Input ~ 0
-постоянка_мк
-Text GLabel 4900 2900 2    50   Input ~ 0
-тип_питания
 Connection ~ 3050 3600
 Wire Wire Line
 	3050 3600 3050 4650
+Text HLabel 5450 2600 2    50   Input ~ 0
+Vout
+Text HLabel 1800 3800 0    50   Input ~ 0
+KEY_V_MK
+Text HLabel 4900 2900 2    50   Input ~ 0
+TYPE_V
 $EndSCHEMATC
